File: hardware/malenki-rx/malenki-rx.kicad_pcb (KiCad board)
At the start: 4 copper layers, 19 x 32 mm, 52 parts, among them J2 Conn_01x08_Male, J3 Conn_01x02, J4 Conn_03x06, U1 A7105, U2 AP2204RA-3.3TRG1, U3 ATTiny1616-MNR, Y1 16mhz Seiko Epson Q24FA20H005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

Commit message: Cleanup old BOM Add a very important crab logo
Parts:
- added REF**: Crab, new-moop-items:Crab, B.Cu at (100.0, 69.5)

Commit message: Fix the crab
Parts:
- moved REF** 2.02 mm to (101.8, 68.5)
Changed lines of the file:
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@@
 	(footprint "new-moop-items:Crab"
 		(layer "B.Cu")
-		(at 100 69.5 90)
+		(at 101.75 68.5 90)
 		(property "Reference" "REF**"
 			(at 0 0.5 270)
@@
 		)
 		(fp_line
-			(start 1.875 -1.254)
+			(start 1.875 -0.77)
 			(end 1.875 -0.254)
 			(stroke
@@
 		)
 		(fp_line
-			(start -1.875 -1.254)
+			(start -1.875 -0.77)
 			(end -1.875 -0.254)
 			(stroke
